File: AD2S1205_EVAL.kicad_pcb (KiCad board)
At the start: 2 copper layers, 39 parts, among them J1 SIN, J2 Power, J3 Interface, J4 COS, J5 DEBUG, J6 EXC, Q1 BD135, Q2 BD136, Q3 BD135, Q4 BD136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

Commit message: layout complete
Parts:
- moved J4 67.8 mm to (107.5, 80.5), turned to 180 degrees
- moved J3 52.3 mm to (107.3, 89.5)
- moved R2 50.4 mm to (126.0, 79.9), turned to -90 degrees
- moved J5 49.5 mm to (155.0, 102.2)
- moved C1 48.5 mm to (125.5, 85.5)
- moved C4 43.7 mm to (134.0, 81.5)
- moved C5 43.4 mm to (132.7, 102.8)
- moved R3 43.4 mm to (144.7, 87.7)
- moved U1 43.4 mm to (134.0, 93.0)
- moved Y1 43.1 mm to (140.0, 103.8)
- moved C3 41.0 mm to (145.0, 100.0), turned to 180 degrees
- moved C2 40.0 mm to (141.0, 100.0), turned to 0 degrees
- moved C9 39.5 mm to (134.0, 77.5)
- moved R1 39.4 mm to (144.0, 77.4), turned to 90 degrees
- moved R9 31.7 mm to (141.0, 84.4), turned to 90 degrees
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Connections:
- J2 pad 2: +5V -> GND
- J2 pad 3: GND -> +5V
Routing:
- net +5V: track 0.00 -> 125.5 mm
- net +12V: track 9.78 -> 79.2 mm
- net GND: track 30.2 -> 64.8 mm
- net Net-(J4-Pin_2): track 0.00 -> 31.4 mm
- net Net-(J4-Pin_1): track 0.00 -> 29.2 mm
- net Net-(J1-Pin_1): track 0.00 -> 28.5 mm
- net Net-(J1-Pin_2): track 0.00 -> 26.6 mm
- net /SCLK: track 0.00 -> 24.2 mm
- net /SO: track 0.00 -> 23.5 mm
- net /~{RDVEL}: track 0.00 -> 22.0 mm
- net /~{SAMPLE}: track 0.00 -> 21.3 mm
- net /~{RD}: track 0.00 -> 21.2 mm
- net Net-(J5-Pin_1): track 0.00 -> 18.2 mm
- net Net-(J5-Pin_2): track 0.00 -> 17.4 mm
- net Net-(J5-Pin_3): track 0.00 -> 16.8 mm
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- added copper zone on F.Cu, net GND

Commit message: layout complete
Parts:
- moved J4 1.96 mm to (107.5, 78.5)
- moved C5 1.44 mm to (134.0, 103.5), turned to 0 degrees
Routing:
- net GND: track 64.8 -> 73.7 mm
- net ~{EXC_AMP}: track 32.0 -> 31.1 mm
- net Net-(J4-Pin_2): track 31.4 -> 32.2 mm
- net Net-(J4-Pin_1): track 29.2 -> 30.0 mm
- net Net-(U1-CLKIN): track 12.8 -> 13.4 mm

Commit message: final
Parts:
- moved J4 11.2 mm to (117.0, 84.5)
- moved R2 7.04 mm to (120.0, 83.6)
- moved J1 6.08 mm to (149.0, 77.0)
- moved R6 5.00 mm to (136.0, 67.9)
- moved R3 4.82 mm to (147.0, 83.5), turned to 180 degrees
- moved R1 2.24 mm to (146.0, 78.4)
- moved R4 1.50 mm to (138.0, 68.0)
- moved C1 1.00 mm to (125.5, 86.5)
- moved C7 1.00 mm to (117.5, 71.5), turned to -90 degrees
Routing:
- net +5V: track 125.4 -> 178.0 mm
- net Net-(J4-Pin_2): track 32.2 -> 20.3 mm
- net Net-(J4-Pin_1): track 30.0 -> 18.8 mm
- net /2.5V: track 23.2 -> 33.2 mm
- net GND: track 73.7 -> 66.8 mm
- net Net-(J1-Pin_1): track 28.5 -> 22.1 mm
- net Net-(J1-Pin_2): track 26.6 -> 20.4 mm
- net Net-(U2B--): track 13.7 -> 16.6 mm, vias 1 -> 2
- net ~{RESET}: track 5.91 -> 8.70 mm
- net +12V: track 79.2 -> 78.1 mm
- net ~{EXC_AMP}: track 31.1 -> 30.1 mm
- net Net-(U2A--): track 13.9 -> 13.1 mm
- net Net-(U1-REFBYP): track 5.39 -> 6.05 mm
Other:
- board outline added: 56 x 59 mm
- board text added: "Michał Zychla 2023"
